File: ESP32-DevKitC/esp32-devkitc_template.kicad_pcb (KiCad board)
At the start: 2 copper layers, 84 parts, among them J1 Conn_01x08, J1 Power, J2 Conn_01x07, J2 Digital/PWM, J3 Analog, J3 Conn_01x07, J4 Digital/PWM, J5 Conn_01x02, J6 Conn_01x03_Pin, J7 Conn_01x03_Pin, J8 Conn_01x03_Pin, Q1 IRLZ44N, U2 ESP32_NODEMCU

Commit message: placas
Parts:
- removed C1 (x2), C2 (x2), C3 (x2): C, Capacitor_THT:CP_Radial_D8.0mm_P3.80mm
- removed the C12V1 at (175.1, 150.7)
- removed the C3.3V1 at (175.1, 158.7)
- removed the C5V1 at (174.8, 140.2)
- removed the Cf1 at (173.3, 166.2)
- removed the Cf2 at (178.3, 174.7)
- removed the Cf3 at (178.3, 170.2)
- removed D1 (x2): LED, LED_THT:LED_D3.0mm
- removed D4 (x2): LED2, LED_THT:LED_D3.0mm
- removed the J1 at (66.0, 81.0)
- removed the J1 at (196.5, 81.5)
- removed the J1 at (250.3, 152.8)
- removed the J2 at (187.4, 33.2)
- removed the J2 at (56.9, 32.7)
- removed the J2 at (193.8, 118.1)
- removed the J3 at (219.4, 81.5)
- removed the J3 at (193.8, 151.0)
- removed the J3 at (88.9, 81.0)
- removed J4 (x2): Digital/PWM, Connector_PinSocket_2.54mm:PinSocket_1x08_P2.54mm_Vertical
- removed J5 (x2): Conn_01x02, TerminalBlock_Phoenix:TerminalBlock_Phoenix_MKDS-1,5-2-5.08_1x02_P5.08mm_Horizontal
- removed J6 (x2), J7 (x2), J8 (x2): Conn_01x03_Pin, Connector_PinHeader_2.54mm:PinHeader_1x03_P2.54mm_Vertical
- removed the JCOOLER1 at (250.3, 143.7)
- removed the JDISPLAY1 at (243.3, 133.2)
- removed the JENCODER1 at (193.8, 137.2)
- removed the JFUENTE1 at (42.4, 33.2)
- removed the JFUENTE1 at (174.8, 116.4)
- removed the JFUENTE1 at (172.9, 33.7)
- removed the JIN1 at (242.8, 113.2)
- removed JMOT0 (x2), JMOT1 (x2), JMOT2 (x2): Conn_01x04_Pin, Connector_PinSocket_2.54mm:PinSocket_1x04_P2.54mm_Vertical
- removed JOUT1 (x2): Conn_01x02, Connector_PinSocket_2.54mm:PinSocket_1x02_P2.54mm_Vertical
- removed the JSD1 at (250.3, 138.3)
- removed MOTX1 (x2), MOTY1 (x2), MOTZ1 (x2): Pololu_Breakout_A4988, Module:Pololu_Breakout-16_15.2x20.3mm
- removed Q1 (x2): IRLZ44N, Package_TO_SOT_THT:TO-220-3_Vertical
- removed R1 (x2): 330R, Resistor_THT:R_Axial_DIN0309_L9.0mm_D3.2mm_P12.70mm_Horizontal
- removed R2 (x2): 1800R, Resistor_THT:R_Axial_DIN0309_L9.0mm_D3.2mm_P12.70mm_Horizontal
- removed R3 (x2): 10R, Resistor_THT:R_Axial_DIN0309_L9.0mm_D3.2mm_P12.70mm_Horizontal
- removed R4 (x2): 10k, Resistor_THT:R_Axial_DIN0309_L9.0mm_D3.2mm_P12.70mm_Horizontal
- removed the U2 at (220.5, 142.7)
- moved Cf1 89.9 mm to (118.8, 116.1)
- moved J3 89.9 mm to (139.3, 100.9)
- moved JIN1 89.9 mm to (188.3, 63.1)
- moved JSD1 89.9 mm to (195.8, 88.2)
- moved J1 89.9 mm to (195.8, 102.7)
- moved J2 89.9 mm to (139.3, 68.0)
- moved JCOOLER1 89.9 mm to (195.8, 93.6)
- moved JDISPLAY1 89.9 mm to (188.8, 83.1)
- moved JENCODER1 89.9 mm to (139.3, 87.1)
- moved JFUENTE1 89.9 mm to (120.3, 66.3)
- moved C12V1 89.9 mm to (120.6, 100.6)
- moved C3.3V1 89.9 mm to (120.6, 108.6)
- moved C5V1 89.9 mm to (120.3, 90.1)
- moved Cf2 89.9 mm to (123.8, 124.6)
- moved Cf3 89.9 mm to (123.8, 120.1)
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Routing:
- net (no net): track 1154.7 -> 0.00 mm, vias 20 -> 0
- net +5V: track 875.8 -> 256.5 mm, vias 8 -> 2
- net +12V: track 696.7 -> 179.8 mm, vias 8 -> 0
- net +3V3: track 216.6 -> 108.3 mm
- net /RX: track 94.3 -> 47.1 mm
- net /MOSI: track 69.8 -> 34.9 mm, vias 4 -> 2
- net /TX: track 67.8 -> 33.9 mm
- net GND: track 32.5 -> 0.00 mm, vias 8 -> 0
- net /CS: track 44.1 -> 22.0 mm
- net /MISO: track 41.9 -> 20.9 mm
- net /SD1: track 40.3 -> 20.2 mm
- net /GPIO4: track 40.3 -> 20.2 mm
- net /SDCLK: track 40.3 -> 20.2 mm
- net /GPIO15: track 40.3 -> 20.2 mm
- net /GPI016: track 40.3 -> 20.2 mm
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