File: ARD-MOTORES/ARD-MOTORES2.kicad_pcb (KiCad board)
At the start: 2 copper layers, 26 parts, among them J1 Power, J2 Digital/PWM, J3 Analog, J4 Digital/PWM, J5 Conn_01x02, J6 Conn_01x03_Pin, J7 Conn_01x03_Pin, J8 Conn_01x03_Pin, Q1 IRLZ44N

Commit message: a
Connections:
- J6 pad 3: /7 -> /*9
- J7 pad 3: /*9 -> /8
- J8 pad 3: /8 -> /7
- MOTX1 pad 16: /13 -> /*3
- MOTY1 pad 16: /*10 -> /*6
- MOTZ1 pad 15: /*3 -> /*10
Changed lines of the file:
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@@
 			(layers "*.Cu" "*.Mask")
 			(remove_unused_layers no)
-			(net 11 "/13")
+			(net 24 "/*3")
 			(pinfunction "DIR")
 			(pintype "input")
@@
 			(layers "*.Cu" "*.Mask")
 			(remove_unused_layers no)
-			(net 18 "/*9")
+			(net 14 "/8")
 			(pinfunction "Pin_3")
 			(pintype "passive")
@@
 			(layers "*.Cu" "*.Mask")
 			(remove_unused_layers no)
-			(net 17 "/*10")
+			(net 21 "/*6")
 			(pinfunction "DIR")
 			(pintype "input")
@@
 			(layers "*.Cu" "*.Mask")
 			(remove_unused_layers no)
-			(net 14 "/8")
+			(net 15 "/7")
 			(pinfunction "Pin_3")
 			(pintype "passive")
@@
 			(layers "*.Cu" "*.Mask")
 			(remove_unused_layers no)
-			(net 15 "/7")
+			(net 18 "/*9")
 			(pinfunction "Pin_3")
 			(pintype "passive")
@@
 			(layers "*.Cu" "*.Mask")
 			(remove_unused_layers no)
-			(net 24 "/*3")
+			(net 17 "/*10")
 			(pinfunction "STEP")
 			(pintype "input")

Commit message: a
Connections:
- MOTX1 pad 15: /12 -> /2
- MOTX1 pad 16: /*3 -> /*5
- MOTY1 pad 15: /*11 -> /*3
- MOTZ1 pad 15: /*10 -> /4
- MOTZ1 pad 16: /2 -> /7
Changed lines of the file:
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@@
 		)
 		(property ki_fp_filters "Connector*:*_1x??_*")
-		(sheetname "Raíz")
+		(sheetname "Root")
 		(sheetfile "ARD-MOTORES2.kicad_sch")
 		(attr through_hole)
@@
 		)
 		(property ki_fp_filters "Connector*:*_1x??_*")
-		(sheetname "Raíz")
+		(sheetname "Root")
 		(sheetfile "ARD-MOTORES2.kicad_sch")
 		(attr through_hole)
@@
 		)
 		(property ki_fp_filters "Connector*:*_1x??_*")
-		(sheetname "Raíz")
+		(sheetname "Root")
 		(sheetfile "ARD-MOTORES2.kicad_sch")
 		(attr through_hole)
@@
 		)
 		(property ki_fp_filters "Connector*:*_1x??_*")
-		(sheetname "Raíz")
+		(sheetname "Root")
 		(sheetfile "ARD-MOTORES2.kicad_sch")
 		(attr through_hole)
@@
 		)
 		(property ki_fp_filters "Connector*:*_1x??_*")
-		(sheetname "Raíz")
+		(sheetname "Root")
 		(sheetfile "ARD-MOTORES2.kicad_sch")
 		(attr through_hole)
@@
 		)
 		(property ki_fp_filters "Pololu*Breakout*15.2x20.3mm*")
-		(sheetname "Raíz")
+		(sheetname "Root")
 		(sheetfile "ARD-MOTORES2.kicad_sch")
 		(attr through_hole)
@@
 			(layers "*.Cu" "*.Mask")
 			(remove_unused_layers no)
-			(net 12 "/12")
+			(net 20 "/2")
 			(pinfunction "STEP")
 			(pintype "input")
@@
 			(layers "*.Cu" "*.Mask")
 			(remove_unused_layers no)
-			(net 24 "/*3")
+			(net 22 "/*5")
 			(pinfunction "DIR")
 			(pintype "input")
@@
 		)
 		(property ki_fp_filters "Connector*:*_1x??_*")
-		(sheetname "Raíz")
+		(sheetname "Root")
 		(sheetfile "ARD-MOTORES2.kicad_sch")
 		(attr through_hole)
@@
 		)
 		(property ki_fp_filters "Connector*:*_1x??_*")
-		(sheetname "Raíz")
+		(sheetname "Root")
 		(sheetfile "ARD-MOTORES2.kicad_sch")
 		(attr through_hole)
@@
 		)
 		(property ki_fp_filters "C_*")
-		(sheetname "Raíz")
+		(sheetname "Root")
 		(sheetfile "ARD-MOTORES2.kicad_sch")
 		(attr through_hole)
@@
 		)
 		(property ki_fp_filters "LED* LED_SMD:* LED_THT:*")
-		(sheetname "Raíz")
+		(sheetname "Root")
 		(sheetfile "ARD-MOTORES2.kicad_sch")
 		(attr through_hole)
@@
 		)
 		(property ki_fp_filters "Connector*:*_1x??_*")
-		(sheetname "Raíz")
+		(sheetname "Root")
 		(sheetfile "ARD-MOTORES2.kicad_sch")
 		(attr through_hole)
@@
 		)
 		(property ki_fp_filters "R_*")
-		(sheetname "Raíz")
+		(sheetname "Root")
 		(sheetfile "ARD-MOTORES2.kicad_sch")
 		(attr through_hole)
@@
 		)
 		(property ki_fp_filters "Pololu*Breakout*15.2x20.3mm*")
-		(sheetname "Raíz")
+		(sheetname "Root")
 		(sheetfile "ARD-MOTORES2.kicad_sch")
 		(attr through_hole)
@@
 			(layers "*.Cu" "*.Mask")
 			(remove_unused_layers no)
-			(net 16 "/*11")
+			(net 24 "/*3")
 			(pinfunction "STEP")
 			(pintype "input")
@@
 		)
 		(property ki_fp_filters "LED* LED_SMD:* LED_THT:*")
-		(sheetname "Raíz")
+		(sheetname "Root")
 		(sheetfile "ARD-MOTORES2.kicad_sch")
 		(attr through_hole)
@@
 		)
 		(property ki_fp_filters "R_*")
-		(sheetname "Raíz")
+		(sheetname "Root")
 		(sheetfile "ARD-MOTORES2.kicad_sch")
 		(attr through_hole)
@@
 		)
 		(property ki_fp_filters "Connector*:*_1x??_*")
-		(sheetname "Raíz")
+		(sheetname "Root")
 		(sheetfile "ARD-MOTORES2.kicad_sch")
 		(attr through_hole)
@@
 		)
 		(property ki_fp_filters "Connector*:*_1x??_*")
-		(sheetname "Raíz")
+		(sheetname "Root")
 		(sheetfile "ARD-MOTORES2.kicad_sch")
 		(attr through_hole)
@@
 		)
 		(property ki_fp_filters "Connector*:*_1x??_*")
-		(sheetname "Raíz")
+		(sheetname "Root")
 		(sheetfile "ARD-MOTORES2.kicad_sch")
 		(attr through_hole)
@@
 		)
 		(property ki_fp_filters "R_*")
-		(sheetname "Raíz")
+		(sheetname "Root")
 		(sheetfile "ARD-MOTORES2.kicad_sch")
 		(attr through_hole)
@@
 		)
 		(property ki_fp_filters "Connector*:*_1x??_*")
-		(sheetname "Raíz")
+		(sheetname "Root")
 		(sheetfile "ARD-MOTORES2.kicad_sch")
 		(attr through_hole)
@@
 		)
 		(property ki_fp_filters "TO?220*")
-		(sheetname "Raíz")
+		(sheetname "Root")
 		(sheetfile "ARD-MOTORES2.kicad_sch")
 		(attr through_hole)
@@
 		)
 		(property ki_fp_filters "R_*")
-		(sheetname "Raíz")
+		(sheetname "Root")
 		(sheetfile "ARD-MOTORES2.kicad_sch")
 		(attr through_hole)
@@
 		)
 		(property ki_fp_filters "Connector*:*_1x??_*")
-		(sheetname "Raíz")
+		(sheetname "Root")
 		(sheetfile "ARD-MOTORES2.kicad_sch")
 		(attr through_hole)
@@
 		)
 		(property ki_fp_filters "Pololu*Breakout*15.2x20.3mm*")
-		(sheetname "Raíz")
+		(sheetname "Root")
 		(sheetfile "ARD-MOTORES2.kicad_sch")
 		(attr through_hole)
@@
 			(layers "*.Cu" "*.Mask")
 			(remove_unused_layers no)
-			(net 17 "/*10")
+			(net 19 "/4")
 			(pinfunction "STEP")
 			(pintype "input")
@@
 			(layers "*.Cu" "*.Mask")
 			(remove_unused_layers no)
-			(net 20 "/2")
+			(net 15 "/7")
 			(pinfunction "DIR")
 			(pintype "input")
@@
 		)
 		(property ki_fp_filters "C_*")
-		(sheetname "Raíz")
+		(sheetname "Root")
 		(sheetfile "ARD-MOTORES2.kicad_sch")
 		(attr through_hole)
@@
 		)
 		(property ki_fp_filters "C_*")
-		(sheetname "Raíz")
+		(sheetname "Root")
 		(sheetfile "ARD-MOTORES2.kicad_sch")
 		(attr through_hole)

Commit message: b
Parts:
- JFUENTE1: footprint TerminalBlock:TerminalBlock_Xinya_XY308-2.54-4P_1x04_P2.54mm_Horizontal -> TerminalBlock_Phoenix:TerminalBlock_Phoenix_MKDS-1,5-4_1x04_P5.00mm_Horizontal
- moved Q1 80.8 mm to (144.5, 90.5), turned to -90 degrees
- moved J5 80.5 mm to (151.8, 108.5)
- moved C1 66.6 mm to (216.5, 94.5), turned to 0 degrees
- moved D4 63.5 mm to (152.0, 96.8)
- moved R2 54.1 mm to (159.8, 81.5), turned to 180 degrees
- moved R4 52.7 mm to (163.3, 74.0)
- moved C2 43.7 mm to (193.2, 94.5), turned to 0 degrees
- moved J6 25.3 mm to (193.5, 65.4)
- moved R3 24.0 mm to (175.3, 66.0), turned to 180 degrees
- moved C3 23.8 mm to (169.7, 94.5), turned to 0 degrees
- moved J8 16.8 mm to (181.0, 65.5)
- moved J7 15.3 mm to (187.5, 65.5)
- moved D1 1.50 mm to (157.5, 59.0)
- moved R1 0.50 mm to (159.0, 76.8)
Connections:
- J7 pad 3: /8 -> /*11
- J8 pad 3: /7 -> /12
- R3 pad 1: /*5 -> /13
Routing:
- net +5V: track 181.5 -> 0.00 mm, vias 2 -> 0
- net +12V: track 168.6 -> 41.5 mm, vias 4 -> 0
- net Net-(D4-K): track 68.7 -> 6.77 mm
- net /8: track 59.3 -> 0.00 mm, vias 2 -> 0
- net Net-(Q1-G): track 53.7 -> 0.00 mm
- net /7: track 53.1 -> 0.00 mm, vias 2 -> 0
- net /*3: track 42.5 -> 0.00 mm, vias 2 -> 0
- net /2: track 39.5 -> 0.00 mm, vias 2 -> 0
- net /*11: track 38.3 -> 0.00 mm
- net /*9: track 37.4 -> 0.96 mm, vias 2 -> 0
- net /*10: track 34.8 -> 0.00 mm
- net /12: track 27.5 -> 0.00 mm
- net GND: track 16.2 -> 0.00 mm, vias 4 -> 0
- net /13: track 23.9 -> 7.79 mm
- net /TX/1: track 11.0 -> 0.00 mm
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Other:
- board text added: "${REFERENCE}"
