File: ARD-MOTORES/ARD-MOTORES2.kicad_sch (KiCad schematic)
At the start: 26 parts, among them J1 Power, J2 Digital/PWM, J3 Analog, J4 Digital/PWM, J5 Conn_01x02, J6 Conn_01x03_Pin, J7 Conn_01x03_Pin, J8 Conn_01x03_Pin, Q1 IRLZ44N

Commit message: cpu_map
Connections:
- net *10: now also J6.3 (Pin_3); no longer MOTY1.16 (DIR)
- net *11: now also J8.3 (Pin_3); no longer MOTY1.15 (STEP)
- net *3: now also MOTY1.15 (STEP); no longer MOTZ1.15 (STEP)
- net *5: now also MOTX1.16 (DIR); no longer R3.1
- net *6: now also MOTY1.16 (DIR)
- net 12: now also R3.1; no longer MOTX1.15 (STEP)
- net 13: no longer MOTX1.16 (DIR)
- net 2: now also MOTX1.15 (STEP); no longer MOTZ1.16 (DIR)
- net 4: now also MOTZ1.15 (STEP)
- net 7: now also MOTZ1.16 (DIR); no longer J6.3 (Pin_3)
- net 8: no longer J8.3 (Pin_3)
Changed lines of the file:
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@@
 	(polyline
 		(pts
-			(xy 237.49 115.57) (xy 237.49 85.09)
+			(xy 237.49 116.84) (xy 237.49 85.09)
 		)
 		(stroke
@@
 	(polyline
 		(pts
-			(xy 237.49 143.51) (xy 237.49 115.57)
+			(xy 237.49 143.51) (xy 237.49 116.84)
 		)
 		(stroke
@@
 	(polyline
 		(pts
-			(xy 285.75 115.57) (xy 237.49 115.57)
+			(xy 285.75 116.84) (xy 237.49 116.84)
 		)
 		(stroke
@@
 		)
 	)
-	(label "*10"
+	(label "*6"
 		(at 180.34 45.72 0)
 		(fields_autoplaced yes)
@@
 		)
 	)
-	(label "8"
+	(label "*11"
 		(at 279.4 106.68 0)
 		(fields_autoplaced yes)
@@
 		)
 	)
-	(label "7"
+	(label "*10"
 		(at 255.27 109.22 0)
 		(fields_autoplaced yes)
@@
 		)
 	)
-	(label "*5"
+	(label "12"
 		(at 172.72 119.38 0)
 		(fields_autoplaced yes)
@@
 		)
 	)
-	(label "*3"
+	(label "4"
 		(at 226.06 41.91 0)
 		(fields_autoplaced yes)
@@
 		)
 	)
-	(label "2"
+	(label "7"
 		(at 226.06 44.45 0)
 		(fields_autoplaced yes)
@@
 		)
 	)
-	(label "*11"
+	(label "*3"
 		(at 180.34 43.18 0)
 		(fields_autoplaced yes)
@@
 		)
 	)
-	(label "13"
+	(label "*5"
 		(at 135.89 45.72 0)
 		(fields_autoplaced yes)
@@
 		)
 	)
-	(label "12"
+	(label "2"
 		(at 135.89 43.18 0)
 		(fields_autoplaced yes)

Commit message: a
Connections:
- net *10: now also MOTZ1.15 (STEP); no longer J6.3 (Pin_3)
- net *11: now also MOTY1.15 (STEP); no longer J8.3 (Pin_3)
- net *3: now also MOTX1.16 (DIR); no longer MOTY1.15 (STEP)
- net *5: now also R3.1; no longer MOTX1.16 (DIR)
- net *9: now also J6.3 (Pin_3); no longer J7.3 (Pin_3)
- net 12: now also MOTX1.15 (STEP); no longer R3.1
- net 2: now also MOTZ1.16 (DIR); no longer MOTX1.15 (STEP)
- net 4: no longer MOTZ1.15 (STEP)
- net 7: now also J8.3 (Pin_3); no longer MOTZ1.16 (DIR)
- net 8: now also J7.3 (Pin_3)
Changed lines of the file:
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@@
 		)
 	)
-	(label "*9"
+	(label "8"
 		(at 267.97 109.22 0)
 		(fields_autoplaced yes)
@@
 		)
 	)
-	(label "*11"
+	(label "7"
 		(at 279.4 106.68 0)
 		(fields_autoplaced yes)
@@
 		)
 	)
-	(label "*10"
+	(label "*9"
 		(at 255.27 109.22 0)
 		(fields_autoplaced yes)
@@
 		)
 	)
-	(label "12"
+	(label "*5"
 		(at 172.72 119.38 0)
 		(fields_autoplaced yes)
@@
 		)
 	)
-	(label "4"
+	(label "*10"
 		(at 226.06 41.91 0)
 		(fields_autoplaced yes)
@@
 		)
 	)
-	(label "7"
+	(label "2"
 		(at 226.06 44.45 0)
 		(fields_autoplaced yes)
@@
 		)
 	)
-	(label "*3"
+	(label "*11"
 		(at 180.34 43.18 0)
 		(fields_autoplaced yes)
@@
 		)
 	)
-	(label "*5"
+	(label "*3"
 		(at 135.89 45.72 0)
 		(fields_autoplaced yes)
@@
 		)
 	)
-	(label "2"
+	(label "12"
 		(at 135.89 43.18 0)
 		(fields_autoplaced yes)

Commit message: a
Connections:
- net *10: no longer MOTZ1.15 (STEP)
- net *11: no longer MOTY1.15 (STEP)
- net *3: now also MOTY1.15 (STEP); no longer MOTX1.16 (DIR)
- net *5: now also MOTX1.16 (DIR)
- net 12: no longer MOTX1.15 (STEP)
- net 2: now also MOTX1.15 (STEP); no longer MOTZ1.16 (DIR)
- net 4: now also MOTZ1.15 (STEP)
- net 7: now also MOTZ1.16 (DIR)
Changed lines of the file:
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@@
 		)
 	)
-	(label "*10"
+	(label "4"
 		(at 226.06 41.91 0)
 		(fields_autoplaced yes)
@@
 		)
 	)
-	(label "2"
+	(label "7"
 		(at 226.06 44.45 0)
 		(fields_autoplaced yes)
@@
 		)
 	)
-	(label "*11"
+	(label "*3"
 		(at 180.34 43.18 0)
 		(fields_autoplaced yes)
@@
 		)
 	)
-	(label "*3"
+	(label "*5"
 		(at 135.89 45.72 0)
 		(fields_autoplaced yes)
@@
 		)
 	)
-	(label "12"
+	(label "2"
 		(at 135.89 43.18 0)
 		(fields_autoplaced yes)

Commit message: b
Connections:
- net *11: now also J7.3 (Pin_3)
- net *5: no longer R3.1
- net 12: now also J8.3 (Pin_3)
- net 13: now also R3.1
- net 7: no longer J8.3 (Pin_3)
- net 8: no longer J7.3 (Pin_3)
Changed lines of the file:
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@@
 		)
 	)
-	(label "8"
+	(label "*11"
 		(at 267.97 109.22 0)
 		(fields_autoplaced yes)
@@
 		)
 	)
-	(label "7"
+	(label "12"
 		(at 279.4 106.68 0)
 		(fields_autoplaced yes)
@@
 		)
 	)
-	(label "*5"
+	(label "13"
 		(at 172.72 119.38 0)
 		(fields_autoplaced yes)
