File: ARD-MOTORES/placa motores.kicad_sch (KiCad schematic)
At the start: 24 parts, among them J1 Power, J2 Digital/PWM, J3 Analog, J4 Digital/PWM, J5 Conn_01x02, Q1 LFRZ44

Commit message: placa motores
Parts:
- removed JLIMX, JLIMY, JLIMZ: 02x02, symbol Connector_Generic:Conn_02x02_Top_Bottom
- removed Q1: LFRZ44, Package_TO_SOT_THT:TO-126-3_Vertical, symbol Transistor_BJT:BF457
- added D4, D5: LED, LED_THT:LED_D5.0mm, symbol Device:LED
- added J6: JLIMX, Connector_PinHeader_2.54mm:PinHeader_1x02_P2.54mm_Vertical, symbol Connector_Generic:Conn_01x02
- added J7: JLIMY, Connector_PinHeader_2.54mm:PinHeader_1x02_P2.54mm_Vertical, symbol Connector_Generic:Conn_01x02
- added J8: JLIMZ, Connector_PinHeader_2.54mm:PinHeader_1x02_P2.54mm_Vertical, symbol Connector_Generic:Conn_01x02
- added Q1: IRLZ44N, Package_TO_SOT_THT:TO-220-3_Vertical, symbol Transistor_FET:IRLZ44N
- added R2, R3: R, Resistor_THT:R_Axial_DIN0414_L11.9mm_D4.5mm_P15.24mm_Horizontal, symbol Device:R
- C1, C2, C3: footprint (none) -> Capacitor_THT:CP_Radial_D6.3mm_P2.50mm
- D1: footprint (none) -> LED_THT:LED_D5.0mm
- D2, D3: footprint (none) -> Diode_THT:D_DO-15_P12.70mm_Horizontal
- J5: footprint (none) -> Connector_PinHeader_2.54mm:PinHeader_1x02_P2.54mm_Vertical
- JFUENTE1: renamed from JFUENTE; footprint (none) -> TerminalBlock_Phoenix:TerminalBlock_Phoenix_MKDS-1,5-4_1x04_P5.00mm_Horizontal
- JMOT0, JMOT1, JMOT2: footprint (none) -> Connector_PinHeader_2.54mm:PinHeader_1x04_P2.54mm_Vertical
- R1: footprint (none) -> Resistor_THT:R_Axial_DIN0414_L11.9mm_D4.5mm_P15.24mm_Horizontal
- out1: renamed from out; footprint (none) -> Connector_PinHeader_2.54mm:PinHeader_1x04_P2.54mm_Vertical
- renumbered MOTX to MOTX1, MOTY to MOTY1, MOTZ to MOTZ1
Connections:
- net *10: now also J7.2 (Pin_2)
- net *11: now also Q1.1 (G)
- net *3: now also MOTZ1.15 (STEP); no longer MOTY1.15 (STEP)
- net *5: now also MOTY1.16 (DIR); no longer MOTX1.16 (DIR)
- net *6: now also MOTX1.15 (STEP); no longer MOTY1.16 (DIR)
- net *9: now also J6.2 (Pin_2)
- net +12V: now also R1.1, Q1.2 (D)
- net +3V3: now also R3.1
- net +5V: now also R2.1; no longer R1.1
- net 12: now also J8.2 (Pin_2)
- net 2: now also MOTZ1.16 (DIR); no longer MOTX1.15 (STEP)
- net 4: now also MOTY1.15 (STEP); no longer MOTZ1.15 (STEP)
- net 7: now also MOTX1.16 (DIR); no longer MOTZ1.16 (DIR)
- net GND: now also D4.1 (K), D5.1 (K), J6.1 (Pin_1), J7.1 (Pin_1), J8.1 (Pin_1)
- net at MOTY1.13 (~{RESET}): now also MOTY1.14 (~{SLEEP})
- net at J5.2 (Pin_2): now also Q1.3 (S)
- net at MOTZ1.13 (~{RESET}): now also MOTZ1.14 (~{SLEEP})
- net at MOTX1.13 (~{RESET}): now also MOTX1.14 (~{SLEEP})
- new net: D5.2 (A), R3.2
- new net: D4.2 (A), R2.2
Other:
- moved on the sheet: D1, JFUENTE1, R1
